Commit message: 系统状态话题确定，反馈适配，模型修改bug

File: src/arm_model/urdf/arm.urdf (robot description, URDF)
Before this commit: robot arm, 10 links, 9 joints
Joints:
- removed joint leftarm_joint1
- removed joint leftarm_joint2
- removed joint leftarm_joint3
- removed joint leftarm_joint4
- removed joint leftarm_joint5
- removed joint leftarm_joint6
- removed joint leftarm_joint7
- added joint armjoint1: type revolute, parent base_link, child leftarm_link1, origin xyz=0 0 0.3 rpy=0 0 0, axis 0 0 1, limit lower=-1.57 upper=1.57 effort=0 velocity=0
- added joint armjoint2: type revolute, parent leftarm_link1, child leftarm_link2, origin xyz=0 0 0 rpy=-1.5708 0 0, axis 0 0 1, limit lower=-1.57 upper=1.57 effort=0 velocity=0
- added joint armjoint3: type revolute, parent leftarm_link2, child leftarm_link3, origin xyz=0 -0.4495 0 rpy=1.5708 0 0, axis 0 0 1, limit lower=-1.57 upper=1.57 effort=0 velocity=0
- added joint armjoint4: type revolute, parent leftarm_link3, child leftarm_link4, origin xyz=-0.03 0 0 rpy=-1.5708 0 0, axis 0 0 1, limit lower=-1.57 upper=1.57 effort=0 velocity=0
- added joint armjoint5: type revolute, parent leftarm_link4, child leftarm_link5, origin xyz=0.03 -0.4495 0 rpy=1.5708 0 0, axis 0 0 1, limit lower=-1.57 upper=1.57 effort=0 velocity=0
- added joint armjoint6: type revolute, parent leftarm_link5, child leftarm_link6, origin xyz=0 0 0 rpy=-1.5708 0 0, axis 0 0 1, limit lower=-1.57 upper=1.57 effort=0 velocity=0
- added joint armjoint7: type revolute, parent leftarm_link6, child leftarm_link7, origin xyz=0 0 0 rpy=1.5708 0 0, axis 0 0 1, limit lower=-1.57 upper=1.57 effort=0 velocity=0
- joint griper_joint1: origin xyz=0.19797 0.027 0.00015 rpy=-3.1416 0 1.5708 -> xyz=-0.19797 -0.027 0.00015 rpy=-3.1416 0 -1.5708
- joint griper_joint2: origin xyz=0.19797 -0.027 0.00015 rpy=0 0 -1.5708 -> xyz=-0.19797 0.027 0.00015 rpy=0 0 1.5708
